File: RedPill.kicad_pcb (KiCad board)
At the start: 4 copper layers, 20.4 x 50.9 mm, 48 parts, among them J1 Conn_01x20, J2 Conn_01x20, J3 USB_C_Receptacle_USB2.0, J4 TagConnect_TC2030_SWD, J5 Conn_01x04, J6 Micro_SD_Card, SW1 SW_Push, U1 STM32F722RETx, U2 SRV05-4, U3 XC6206PxxxMR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

Commit message: Attach 5V pin to input capacitor
Other:
- rule pad_to_mask_clearance: 0.05 -> 0
Changed lines of the file:
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@@
     (thickness 1.6)
     (drawings 64)
-    (tracks 638)
+    (tracks 637)
     (zones 0)
     (modules 48)
@@
   )
   (setup
-    (last_trace_width 0.25)
+    (last_trace_width 0.5)
     (user_trace_width 0.09)
     (user_trace_width 0.127)
@@
     (pad_size 1.524 1.524)
     (pad_drill 0.762)
-    (pad_to_mask_clearance 0.05)
+    (pad_to_mask_clearance 0)
+    (pad_to_paste_clearance_ratio -0.05)
     (aux_axis_origin 0 0)
     (grid_origin 100 100)
@@
     (pcbplotparams
       (layerselection 0x010fc_ffffffff)
-      (usegerberextensions false)
+      (usegerberextensions true)
       (usegerberattributes true)
       (usegerberadvancedattributes true)
-      (creategerberjobfile true)
+      (creategerberjobfile false)
       (excludeedgelayer true)
       (linewidth 0.100000)
@@
       (outputformat 1)
       (mirror false)
-      (drillshape 1)
+      (drillshape 0)
       (scaleselection 1)
       (outputdirectory ""))
@@
   (segment (start 108.5 113.65) (end 107.725 114.425) (width 0.25) (layer F.Cu) (net 10))
   (segment (start 107.935 116.535) (end 107.725 116.325) (width 0.25) (layer F.Cu) (net 10))
-  (segment (start 103.535 113.285) (end 103.525 113.275) (width 0.5) (layer F.Cu) (net 11))
   (segment (start 105 113.325) (end 104.96 113.285) (width 0.5) (layer F.Cu) (net 11))
   (segment (start 105 114.5125) (end 105 113.325) (width 0.5) (layer F.Cu) (net 11))
-  (segment (start 104.96 113.285) (end 103.535 113.285) (width 0.5) (layer F.Cu) (net 11))
+  (segment (start 105.175 113.25) (end 103.75 113.25) (width 0.5) (layer F.Cu) (net 11))
   (segment (start 105.3 113.285) (end 104.96 113.285) (width 0.5) (layer F.Cu) (net 11))
   (segment (start 106.5 114.6) (end 106.5 114.475) (width 0.25) (layer F.Cu) (net 11))
   (segment (start 106.5 114.475) (end 105.3 113.275) (width 0.25) (layer F.Cu) (net 11))
   (via (at 103.6 114) (size 0.45) (drill 0.2) (layers F.Cu B.Cu) (net 11))
-  (segment (start 103.6 113.05) (end 103.6 114) (width 0.5) (layer F.Cu) (net 11))
   (via (at 103.6 114.6) (size 0.45) (drill 0.2) (layers F.Cu B.Cu) (net 11))
   (segment (start 103.6 114) (end 103.6 114.6) (width 0.5) (layer F.Cu) (net 11))
@@
   (segment (start 103.6 115.1) (end 103.6 114.6) (width 1) (layer Power) (net 11))
   (segment (start 107.55 119.05) (end 103.6 115.1) (width 1) (layer Power) (net 11))
+  (segment (start 103.6 114.6) (end 105 114.6) (width 0.5) (layer F.Cu) (net 11))
   (segment (start 106.831713 130.157375) (end 106.831713 130.168287) (width 0.09) (layer F.Cu) (net 12))
   (segment (start 106.831713 130.157375) (end 106.189088 130.8) (width 0.127) (layer F.Cu) (net 12))
